File: PCB_without_Ard/PCB_BLDC.kicad_pcb (KiCad board)
At the start: 2 copper layers, 158.8 x 92.7 mm, 77 parts, among them J1 Ground Terminal, J10 Conn_01x02, J2 Conn_01x03, J3 Conn_01x05, J4 Conn_01x02, J5 Conn_01x03, J6 Conn_01x03, J7 Conn_01x03, J8 Power Terminal, J9 Conn_01x02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

Commit message: PCB: Final Review. Add new Push Button, Change wrong Capacitors Change Routing, Add Mounting Holes
Parts:
- added C30: 1uF, Capacitor_SMD:C_1206_3216Metric_Pad1.33x1.80mm_HandSolder, F.Cu at (46.1, 79.0)
- added R28: 10k, Resistor_SMD:R_1206_3216Metric_Pad1.30x1.75mm_HandSolder, F.Cu at (67.0, 79.1)
- added R29: 10k, Resistor_SMD:R_1206_3216Metric_Pad1.30x1.75mm_HandSolder, F.Cu at (56.9, 79.0)
- added SW3: SW_Push, Button_Switch_THT:SW_PUSH-12mm_Wuerth-430476085716, F.Cu at (58.5, 66.2)
- C14, C15, C16, C17, C18, C19, C20, C21, C22: footprint Capacitor_SMD:C_Elec_5x5.4 -> Capacitor_SMD:C_1206_3216Metric_Pad1.33x1.80mm_HandSolder
- C23, C24, C25: value 470nF -> 470uF; footprint Capacitor_SMD:C_Elec_5x5.4 -> Capacitor_SMD:CP_Elec_16x17.5
- J9: value Conn_01x02 -> Conn_01x04; footprint Connector_PinSocket_2.54mm:PinSocket_1x03_P2.54mm_Vertical -> Connector_PinSocket_2.54mm:PinSocket_1x04_P2.54mm_Vertical
- moved C29 35.1 mm to (46.3, 85.2), turned to 180 degrees
- moved D3 34.5 mm to (98.6, 85.6), turned to 180 degrees
- moved J9 31.5 mm to (80.8, 77.0)
- moved R3 30.4 mm to (91.5, 85.6), turned to 0 degrees
- moved R27 28.0 mm to (57.3, 85.3), turned to 180 degrees
- moved SW1 25.7 mm to (66.5, 107.1)
- moved C6 25.7 mm to (45.5, 113.6)
- moved C7 25.7 mm to (45.5, 106.0)
- moved J4 25.7 mm to (52.5, 108.4)
- moved R16 25.7 mm to (58.6, 106.0)
- moved R17 25.7 mm to (58.6, 113.5)
- moved R26 21.8 mm to (72.7, 88.6)
- moved SW2 15.6 mm to (58.8, 97.5), turned to 180 degrees
- moved R4 11.4 mm to (96.4, 118.9), turned to 90 degrees
- moved C9 7.51 mm to (133.7, 120.4), turned to 270 degrees
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Connections:
- J9 pad 2: /Reset_SW -> /Stop_SW
- J9 pad 3: GND -> /Reset_SW
Routing:
- net /Stop_SW: track 0.00 -> 34.7 mm
- net GND: track 136.7 -> 103.0 mm
- net /VCC_Filtered: track 278.0 -> 260.6 mm
- net /Reset_SW: track 17.9 -> 34.0 mm
- net Net-(R28-Pad1): track 0.00 -> 15.1 mm
- net /L3_Motor: track 77.6 -> 66.5 mm
- net /L3_IS: track 64.2 -> 55.0 mm
- net /L1_Motor: track 68.2 -> 59.8 mm
- net /VCC_5V: track 125.6 -> 118.6 mm
- net Net-(R9-Pad1): track 18.9 -> 24.6 mm
- net Net-(R8-Pad1): track 17.5 -> 23.2 mm
- net /L1_IS: track 59.1 -> 54.7 mm
- net Net-(R26-Pad1): track 15.6 -> 19.7 mm
- net Net-(R11-Pad1): track 16.8 -> 20.8 mm
- net /L2_IS: track 61.4 -> 57.5 mm
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Other:
- board text added: "B | A"
- board text added: "Stop"
- board text added: "Stop Push Button"
- board text removed: "A | B"
