File: PCB_without_Ard/PCB_BLDC.sch (KiCad schematic (older format))
At the start: 72 parts, among them J1 Ground Terminal, J2 Conn_01x03, J3 Conn_01x05, J4 Conn_01x02, J5 Conn_01x04, J6 Conn_01x04, J7 Conn_01x04, J8 Power Terminal, J9 Conn_01x02, Q1 IRF4905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

Commit message: Add Push Button to Reset the System
Parts:
- added C29: 1uF, Capacitor_SMD:C_1206_3216Metric_Pad1.33x1.80mm_HandSolder, symbol Device:C_Small
- added R26, R27: 10k, Resistor_SMD:R_1206_3216Metric_Pad1.30x1.75mm_HandSolder, symbol Device:R_Small
- added SW2: SW_Push, Button_Switch_THT:SW_PUSH-12mm_Wuerth-430476085716, symbol Switch:SW_Push
- J9: footprint Connector_PinSocket_2.54mm:PinSocket_1x02_P2.54mm_Vertical -> Connector_PinSocket_2.54mm:PinSocket_1x03_P2.54mm_Vertical; symbol Connector_Generic:Conn_01x02 -> Connector_Generic:Conn_01x03
Connections:
- net GND: now also J9.3 (Pin_3), C29.2, SW2.1; no longer J9.2 (Pin_2)
- net VCC_5V: now also R26.2
- new net: R26.1, R27.1, SW2.2
- new net Reset_SW: C29.1, J9.2 (Pin_2), R27.2
Other:
- note added: "Reet Push Button"
Changed lines of the file:
@@
 $EndComp
 $Comp
-L Connector_Generic:Conn_01x02 J9
+L Connector_Generic:Conn_01x03 J9
 U 1 1 61BA226F
 P 1350 4050
 F 0 "J9" H 1430 4042 50  0000 L CNN
-F 1 "Conn_01x02" H 800 4150 50  0000 L CNN
-F 2 "Connector_PinSocket_2.54mm:PinSocket_1x02_P2.54mm_Vertical" H 1350 4050 50  0001 C CNN
+F 1 "Conn_01x02" H 1100 3800 50  0000 L CNN
+F 2 "Connector_PinSocket_2.54mm:PinSocket_1x03_P2.54mm_Vertical" H 1350 4050 50  0001 C CNN
 F 3 "~" H 1350 4050 50  0001 C CNN
 	1    1350 4050
 	1    0    0    -1
 $EndComp
-Text Label 950  4050 2    50   ~ 0
+Text Label 950  3950 2    50   ~ 0
 VCC_5V
 $Comp
@@
 	-1   0    0    1
 $EndComp
+$Comp
+L Switch:SW_Push SW2
+U 1 1 6192548F
+P 3200 6150
+F 0 "SW2" V 3246 6102 50  0000 R CNN
+F 1 "SW_Push" V 3155 6102 50  0000 R CNN
+F 2 "Button_Switch_THT:SW_PUSH-12mm_Wuerth-430476085716" H 3200 6350 50  0001 C CNN
+F 3 "~" H 3200 6350 50  0001 C CNN
+	1    3200 6150
+	0    -1   -1   0
+$EndComp
+$Comp
+L Device:R_Small R26
+U 1 1 6195C156
+P 3200 5650
+F 0 "R26" V 3350 5700 50  0000 R CNN
+F 1 "10k" V 3250 5750 50  0000 R CNN
+F 2 "Resistor_SMD:R_1206_3216Metric_Pad1.30x1.75mm_HandSolder" H 3200 5650 50  0001 C CNN
+F 3 "~" H 3200 5650 50  0001 C CNN
+	1    3200 5650
+	-1   0    0    1
+$EndComp
+$Comp
+L Device:R_Small R27
+U 1 1 6195C4AE
+P 3700 5950
+F 0 "R27" V 3850 6000 50  0000 R CNN
+F 1 "10k" V 3750 6050 50  0000 R CNN
+F 2 "Resistor_SMD:R_1206_3216Metric_Pad1.30x1.75mm_HandSolder" H 3700 5950 50  0001 C CNN
+F 3 "~" H 3700 5950 50  0001 C CNN
+	1    3700 5950
+	0    -1   -1   0
+$EndComp
+$Comp
+L Device:C_Small C29
+U 1 1 6195C953
+P 4050 6150
+F 0 "C29" H 3900 6150 50  0000 C CNN
+F 1 "1uF" H 3950 6250 50  0000 C CNN
+F 2 "Capacitor_SMD:C_1206_3216Metric_Pad1.33x1.80mm_HandSolder" H 4050 6150 50  0001 C CNN
+F 3 "~" H 4050 6150 50  0001 C CNN
+	1    4050 6150
+	1    0    0    -1
+$EndComp
+$Comp
+L power:GND #PWR08
+U 1 1 6195CF12
+P 3200 6450
+F 0 "#PWR08" H 3200 6200 50  0001 C CNN
+F 1 "GND" H 3205 6277 50  0000 C CNN
+F 2 "" H 3200 6450 50  0001 C CNN
+F 3 "" H 3200 6450 50  0001 C CNN
+	1    3200 6450
+	1    0    0    -1
+$EndComp
+$Comp
+L power:GND #PWR09
+U 1 1 6195D25A
+P 4050 6450
+F 0 "#PWR09" H 4050 6200 50  0001 C CNN
+F 1 "GND" H 4055 6277 50  0000 C CNN
+F 2 "" H 4050 6450 50  0001 C CNN
+F 3 "" H 4050 6450 50  0001 C CNN
+	1    4050 6450
+	1    0    0    -1
+$EndComp
+Text Label 3200 5300 2    50   ~ 0
+VCC_5V
+Wire Wire Line
+	3200 5300 3200 5550
+Wire Wire Line
+	3200 6350 3200 6450
+Wire Wire Line
+	3200 5750 3200 5950
+Wire Wire Line
+	4050 6450 4050 6250
+Wire Wire Line
+	4050 6050 4050 5950
+Wire Wire Line
+	3200 5950 3600 5950
+Wire Wire Line
+	3800 5950 4050 5950
+Connection ~ 3200 5950
+Connection ~ 4050 5950
+Wire Wire Line
+	4050 5950 4350 5950
+Wire Wire Line
+	950  3950 1150 3950
+Text Label 950  4050 2    50   ~ 0
+Reset_SW
+Text Label 4350 5950 0    50   ~ 0
+Reset_SW
+Wire Notes Line
+	2900 5150 2900 6750
+Wire Notes Line
+	2900 6750 4750 6750
+Wire Notes Line
+	4750 6750 4750 5150
+Wire Notes Line
+	4750 5150 2900 5150
+Text Notes 3500 5100 0    50   ~ 0
+Reet Push Button
 $EndSCHEMATC

Commit message: PCB: Change Position of RC Filt for Hall Sense and Position of Connector
Parts:
- added J10: Conn_01x02, Connector_PinSocket_2.54mm:PinSocket_1x03_P2.54mm_Vertical, symbol Connector_Generic:Conn_01x03
- J5, J6, J7: value Conn_01x04 -> Conn_01x03; footprint Connector_PinSocket_2.54mm:PinSocket_1x04_P2.54mm_Vertical -> Connector_PinSocket_2.54mm:PinSocket_1x03_P2.54mm_Vertical; symbol Connector_Generic:Conn_01x04 -> Connector_Generic:Conn_01x03
Connections:
- net L1_IN: now also J5.1 (Pin_1); no longer J5.2 (Pin_2)
- net L1_INH: now also J5.2 (Pin_2); no longer J5.3 (Pin_3)
- net L1_IS: now also J5.3 (Pin_3); no longer J5.4 (Pin_4)
- net L1_Sense: now also R20.1; no longer R18.1
- net L2_IN: now also J6.1 (Pin_1); no longer J6.2 (Pin_2)
- net L2_INH: now also J6.2 (Pin_2); no longer J6.3 (Pin_3)
- net L2_IS: now also J6.3 (Pin_3); no longer J6.4 (Pin_4)
- net L2_Sense: now also R23.1; no longer R19.1
- net L3_IN: now also J7.1 (Pin_1); no longer J7.2 (Pin_2)
- net L3_INH: now also J7.2 (Pin_2); no longer J7.3 (Pin_3)
- net L3_IS: now also J7.3 (Pin_3); no longer J7.4 (Pin_4)
- net L3_Sense: now also R18.1, R19.1; no longer R20.1, R23.1
- net VCC_5V: now also R18.2, R20.2; no longer R21.2, R23.2
- new net L1_Sense_Filt: C27.1, J10.1 (Pin_1), R21.2
- new net L2_Sense_Filt: C28.1, J10.2 (Pin_2), R23.2
- new net L3_Sense_Filt: C26.1, J10.3 (Pin_3), R19.2
Other:
- note added: "Hall Sensor Connector"
- note added: "L1 Sense Filter"
- note added: "L2 Sense Filter"
- note added: "L3 Sense Filter"
- moved on the sheet: C29, C6, C7, D2, D3, J4, R16, R17, R24, R25, R26, R27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

Commit message: PCB: Final Review. Add new Push Button, Change wrong Capacitors Change Routing, Add Mounting Holes
Parts:
- added C30: 1uF, Capacitor_SMD:C_1206_3216Metric_Pad1.33x1.80mm_HandSolder, symbol Device:C_Small
- added R28, R29: 10k, Resistor_SMD:R_1206_3216Metric_Pad1.30x1.75mm_HandSolder, symbol Device:R_Small
- added SW3: SW_Push, Button_Switch_THT:SW_PUSH-12mm_Wuerth-430476085716, symbol Switch:SW_Push
- C14, C15, C16, C17, C18, C19, C20, C21, C22: footprint Capacitor_SMD:C_Elec_5x5.4 -> Capacitor_SMD:C_1206_3216Metric_Pad1.33x1.80mm_HandSolder
- C23, C24, C25: value 470nF -> 470uF; footprint Capacitor_SMD:C_Elec_5x5.4 -> Capacitor_SMD:CP_Elec_16x17.5; symbol Device:C_Small -> Device:CP_Small
- J9: value Conn_01x02 -> Conn_01x04; footprint Connector_PinSocket_2.54mm:PinSocket_1x03_P2.54mm_Vertical -> Connector_PinSocket_2.54mm:PinSocket_1x04_P2.54mm_Vertical; symbol Connector_Generic:Conn_01x03 -> Connector_Generic:Conn_01x04
Connections:
- net GND: now also J9.4 (Pin_4), C30.2, SW3.1; no longer J9.3 (Pin_3)
- net Reset_SW: now also J9.3 (Pin_3); no longer J9.2 (Pin_2)
- net VCC_5V: now also R28.2
- new net: R28.1, R29.1, SW3.2
- new net Stop_SW: C30.1, J9.2 (Pin_2), R29.2
Other:
- note added: "Reset Push Button"
- note added: "Stop Push Button"
- note removed: "Reet Push Button"
- moved on the sheet: C26, R18, R19
